File: ECAD/Self_Watering_Plant.kicad_sch (KiCad schematic)
At the start: 17 parts, among them J1 Conn_01x02, J2 Conn_01x02, J3 USB_A, J6 USB_A, J7 Conn_01x02, J8 Conn_01x02, J9 Conn_01x03, P1 U262-161N-4BVC11, U11 BCT2028

Commit message: BOM fixed, ready to order
Parts:
- C12, C14: Manufacturer (none) -> Samsung Electro-Mechanics; Manufacturer Number (none) -> CL10A105KO8NNNC
- C13: Manufacturer (none) -> CCTC; Manufacturer Number (none) -> TCC0603X7R103M500CT
- D3, D6: Manufacturer (none) -> Shikues; Manufacturer Number (none) -> RS3ABG
- F1: Manufacturer (none) -> BOURNS; Manufacturer Number (none) -> MF-MSMF110/24X-2
- J1, J2: Manufacturer (none) -> Ningbo Kangnex Elec; Manufacturer Number MF-MSMF110/24X-2 -> WJ127-5.0-2P
- J3, J6: Manufacturer (none) -> MOLEX; Manufacturer Number (none) -> 676432911
- J7, J8: Manufacturer (none) -> JST Sales America; Manufacturer Number (none) -> S2B-XH-A(LF)(SN)
- J9: Manufacturer (none) -> JST Sales America; Manufacturer Number (none) -> S3B-XH-A(LF)(SN)
- P1: Manufacturer (none) -> XKB Connectivity; Manufacturer Number (none) -> U262-161N-4BVC11
- R2, R5: Manufacturer (none) -> YAGEO; Manufacturer Number (none) -> RC0603JR-075K1L
- U11: Manufacturer (none) -> BROADCHIP; Manufacturer Number (none) -> BCT2028EUK33-TR

Commit message: adding production and step files
Parts:
- C12, C14: Manufacturer Samsung Electro-Mechanics -> Samsung Electro-Mechanics; Package (none) -> 0603; Rated Voltage 6.3V -> (none)
- C13: Package (none) -> 0603; Rated Voltage 6.3V -> (none)
- D3, D6: Package (none) -> SMB
- F1: Package (none) -> 1812
- J1, J2: Manufacturer Ningbo Kangnex Elec -> (none); Manufacturer Number WJ127-5.0-2P -> WJ127-5.0-2P; Package (none) -> P=5.0mm
- J3, J6: Package (none) -> Through Hole
- J7, J8, J9: Package (none) -> Through Hole,P=2.5mm
- P1: value U262-161N-4BVC11 -> C-31-M-12; footprint Connector_USB:USB_C_Receptacle_XKB_U262-16XN-4BVC11 -> Connector_USB:USB_C_Receptacle_HRO_TYPE-C-31-M-12; Manufacturer XKB Connectivity -> Korean Hroparts Elec; Package (none) -> SMT
- R2, R5: Manufacturer YAGEO -> UNI-ROYAL(Uniroyal Elec); Manufacturer Number RC0603JR-075K1L -> 0603WAF5101T5E; Package (none) -> 0603
- U11: Package (none) -> SOT-23-5
Connections:
- no-connect marks 0 -> 4
Other:
- sheet Controller ports: added SCL, SDA; removed DH11_IO
- sheet TempAndHumiditySensor ports: added SCL, SDA; removed IO
